File: wifiSens/Schematic/file5A51538F.sch (KiCad schematic (older format))
At the start: 12 parts, among them J2 CONN_01X04, U2 ESP-12E

Commit message: moved to ubuntu
Parts:
- C10: value C -> 100n
Changed lines of the file:
@@
 LIBS:contrib
 LIBS:valves
-LIBS:ESP8266
 LIBS:wifiSens
 LIBS:switches
@@
 P 1850 5000
 F 0 "C10" H 1875 5100 50  0000 L CNN
-F 1 "C" H 1875 4900 50  0000 L CNN
+F 1 "100n" H 1875 4900 50  0000 L CNN
 F 2 "Capacitors_SMD:C_0603_HandSoldering" H 1888 4850 50  0001 C CNN
 F 3 "" H 1850 5000 50  0001 C CNN
